File: 02_PCB/LightspeedLaserDriver/BoostConverter.kicad_sch (KiCad schematic)
At the start: 24 parts, among them IC1 LT8365JMSE, SW1 SW_SPDT

Commit message: feat(pcb): add peripherals to PCB
Parts:
- removed SW1: SW_SPDT, Button_Switch_SMD:SW_SPDT_PCM12, symbol Switch:SW_SPDT
- added SW2: JS202011JAQN, Button_Switch_SMD:SW_DPDT_CK_JS202011JCQN, symbol Switch:SW_Push_DPDT
- D2, D3, D4: value DFLS1150 -> SMD115PBQ-TP; footprint Diode_SMD:D_PowerDI-123 -> CustomFootprints:D_SOD-323HE
- L1: value 10u -> 74438356220; footprint Inductor_SMD:L_Wuerth_HCM-7050 -> Inductor_SMD:L_Wuerth_MAPI-4020
Connections:
- net GND: now also D5.1 (K), SW2.4 (A), SW2.5 (B), SW2.6 (C)
- net VIN: now also SW2.3 (C); no longer R6.1, R7.2
- new net: R6.1, R7.2, SW2.2 (B)
- no-connect marks 0 -> 1
Other:
- note added: "Reference design: 74437324100 (10uH) Available alternative: 74438336100 (10uH, tiny) Available alternative: 74438356150 (15uH) Better alternative: 74438356220 (22uH) Performance alternative: 744393305220 (22uH)"
- moved on the sheet: D5, R6, R7, R8

Commit message: feat(pcb): route all traces
Parts:
- renumbered D2 to D3, D3 to D4, D4 to D5, D5 to D6, R8 to R10, R1 to R3, R2 to R4, R3 to R5, R4 to R6, R5 to R7, R6 to R8, R7 to R9, SW2 to SW1
Connections:
- net FBX: now also RV1.1; no longer RV1.3
- net at R8.1, R9.2, SW1.2 (B): now also SW1.1 (A)
- net at R7.1: now also RV1.3; no longer RV1.1
- no-connect marks 1 -> 0
Other:
- moved on the sheet: RV1
Changed lines of the file:
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@@
+	)
+	(junction
+		(at 252.73 82.55)
+		(diameter 0)
+		(color 0 0 0 0)
 	)
 	(junction
@@
 	)
 	(junction
-		(at 218.44 80.01)
+		(at 218.44 78.74)
 		(diameter 0)
 		(color 0 0 0 0)
@@
 		(color 0 0 0 0)
 	)
-	(no_connect
-		(at 256.54 67.31)
-	)
 	(wire
 		(pts
@@
 	(wire
 		(pts
+			(xy 222.25 83.82) (xy 223.52 83.82)
+		)
+		(stroke
+			(width 0)
+			(type default)
+		)
+	)
+	(wire
+		(pts
 			(xy 218.44 63.5) (xy 218.44 66.04)
 		)
@@
 	(wire
 		(pts
-			(xy 213.36 85.09) (xy 214.63 85.09)
+			(xy 218.44 87.63) (xy 218.44 91.44)
 		)
 		(stroke
@@
 	(wire
 		(pts
+			(xy 223.52 78.74) (xy 218.44 78.74)
+		)
+		(stroke
+			(width 0)
+			(type default)
+		)
+	)
+	(wire
+		(pts
 			(xy 121.92 102.87) (xy 125.73 102.87)
 		)
@@
 	(wire
 		(pts
+			(xy 256.54 66.04) (xy 252.73 66.04)
+		)
+		(stroke
+			(width 0)
+			(type default)
+		)
+	)
+	(wire
+		(pts
 			(xy 154.94 92.71) (xy 154.94 95.25)
 		)
@@
 	(wire
 		(pts
-			(xy 213.36 80.01) (xy 213.36 85.09)
-		)
-		(stroke
-			(width 0)
-			(type default)
-		)
-	)
-	(wire
-		(pts
 			(xy 83.82 102.87) (xy 63.5 102.87)
 		)
@@
 	(wire
 		(pts
-			(xy 218.44 81.28) (xy 218.44 80.01)
+			(xy 252.73 66.04) (xy 252.73 82.55)
 		)
 		(stroke
@@
 	(wire
 		(pts
+			(xy 256.54 67.31) (xy 256.54 66.04)
+		)
+		(stroke
+			(width 0)
+			(type default)
+		)
+	)
+	(wire
+		(pts
 			(xy 252.73 83.82) (xy 252.73 82.55)
 		)
@@
 	(wire
 		(pts
-			(xy 218.44 76.2) (xy 218.44 80.01)
-		)
-		(stroke
-			(width 0)
-			(type default)
-		)
-	)
-	(wire
-		(pts
-			(xy 218.44 80.01) (xy 213.36 80.01)
-		)
-		(stroke
-			(width 0)
-			(type default)
-		)
-	)
-	(wire
-		(pts
 			(xy 121.92 92.71) (xy 154.94 92.71)
 		)
@@
 	(wire
 		(pts
-			(xy 218.44 88.9) (xy 218.44 91.44)
-		)
-		(stroke
-			(width 0)
-			(type default)
-		)
-	)
-	(wire
-		(pts
 			(xy 69.85 114.3) (xy 69.85 115.57)
 		)
@@
 	(wire
 		(pts
+			(xy 218.44 78.74) (xy 218.44 80.01)
+		)
+		(stroke
+			(width 0)
+			(type default)
+		)
+	)
+	(wire
+		(pts
 			(xy 158.75 81.28) (xy 165.1 81.28)
 		)
@@
 	(wire
 		(pts
+			(xy 223.52 83.82) (xy 223.52 78.74)
+		)
+		(stroke
+			(width 0)
+			(type default)
+		)
+	)
+	(wire
+		(pts
 			(xy 184.15 67.31) (xy 184.15 60.96)
 		)
@@
 		(pts
 			(xy 218.44 99.06) (xy 218.44 100.33)
+		)
+		(stroke
+			(width 0)
+			(type default)
+		)
+	)
+	(wire
+		(pts
+			(xy 218.44 76.2) (xy 218.44 78.74)
 		)
 		(stroke
@@
 		(on_board yes)
 		(dnp no)
-		(property "Reference" "D2"
+		(property "Reference" "D3"
 			(at 155.194 75.438 0)
 			(effects
@@
 			(project "LightspeedLaserDriver"
 				(path "/8e13b6ca-3b5b-4f2e-83bc-fdfde26a6699/6c7faaef-a9df-4a02-8e80-f9afae2d6d46"
-					(reference "D2")
+					(reference "D3")
 					(unit 1)
 				)
@@
 		(on_board yes)
 		(dnp no)
-		(property "Reference" "R4"
+		(property "Reference" "R6"
 			(at 221.996 68.326 0)
 			(effects
@@
 			(project "LightspeedLaserDriver"
 				(path "/8e13b6ca-3b5b-4f2e-83bc-fdfde26a6699/6c7faaef-a9df-4a02-8e80-f9afae2d6d46"
-					(reference "R4")
+					(reference "R6")
 					(unit 1)
 				)
@@
 		(dnp no)
 		(fields_autoplaced yes)
-		(property "Reference" "R2"
+		(property "Reference" "R4"
 			(at 157.48 97.7899 0)
 			(effects
@@
 			(project "LightspeedLaserDriver"
 				(path "/8e13b6ca-3b5b-4f2e-83bc-fdfde26a6699/6c7faaef-a9df-4a02-8e80-f9afae2d6d46"
-					(reference "R2")
+					(reference "R4")
 					(unit 1)
 				)
@@
 		(on_board yes)
 		(dnp no)
-		(property "Reference" "R6"
+		(property "Reference" "R8"
 			(at 250.19 86.3599 0)
 			(effects
@@
 			(project ""
 				(path "/8e13b6ca-3b5b-4f2e-83bc-fdfde26a6699/6c7faaef-a9df-4a02-8e80-f9afae2d6d46"
-					(reference "R6")
+					(reference "R8")
 					(unit 1)
 				)
@@
 		(dnp no)
 		(fields_autoplaced yes)
-		(property "Reference" "D4"
+		(property "Reference" "D5"
 			(at 175.5775 54.61 0)
 			(effects
@@
 			(project "LightspeedLaserDriver"
 				(path "/8e13b6ca-3b5b-4f2e-83bc-fdfde26a6699/6c7faaef-a9df-4a02-8e80-f9afae2d6d46"
-					(reference "D4")
+					(reference "D5")
 					(unit 1)
 				)
@@
 		(on_board yes)
 		(dnp no)
-		(property "Reference" "R8"
+		(property "Reference" "R10"
 			(at 262.128 96.774 0)
 			(effects
@@
 			(project "LightspeedLaserDriver"
 				(path "/8e13b6ca-3b5b-4f2e-83bc-fdfde26a6699/6c7faaef-a9df-4a02-8e80-f9afae2d6d46"
-					(reference "R8")
+					(reference "R10")
 					(unit 1)
 				)
@@
 		(dnp no)
 		(fields_autoplaced yes)
-		(property "Reference" "R5"
+		(property "Reference" "R7"
 			(at 220.98 93.9799 0)
 			(effects
@@
 			(project "LightspeedLaserDriver"
 				(path "/8e13b6ca-3b5b-4f2e-83bc-fdfde26a6699/6c7faaef-a9df-4a02-8e80-f9afae2d6d46"
-					(reference "R5")
+					(reference "R7")
 					(unit 1)
 				)
@@
 		(dnp no)
 		(fields_autoplaced yes)
-		(property "Reference" "R3"
+		(property "Reference" "R5"
 			(at 167.64 73.6599 0)
 			(effects
@@
 			(project "LightspeedLaserDriver"
 				(path "/8e13b6ca-3b5b-4f2e-83bc-fdfde26a6699/6c7faaef-a9df-4a02-8e80-f9afae2d6d46"
-					(reference "R3")
+					(reference "R5")
 					(unit 1)
 				)
@@
 		(on_board yes)
 		(dnp no)
-		(property "Reference" "R7"
+		(property "Reference" "R9"
 			(at 261.874 86.36 0)
 			(effects
@@
 			(project "LightspeedLaserDriver"
 				(path "/8e13b6ca-3b5b-4f2e-83bc-fdfde26a6699/6c7faaef-a9df-4a02-8e80-f9afae2d6d46"
-					(reference "R7")
+					(reference "R9")
 					(unit 1)
 				)
@@
 		(dnp no)
 		(fields_autoplaced yes)
-		(property "Reference" "R1"
+		(property "Reference" "R3"
 			(at 72.39 109.2199 0)
 			(effects
@@
 			(project "LightspeedLaserDriver"
 				(path "/8e13b6ca-3b5b-4f2e-83bc-fdfde26a6699/6c7faaef-a9df-4a02-8e80-f9afae2d6d46"
-					(reference "R1")
+					(reference "R3")
 					(unit 1)
 				)
@@
 		(dnp no)
 		(fields_autoplaced yes)
-		(property "Reference" "D5"
+		(property "Reference" "D6"
 			(at 248.92 98.1074 90)
 			(effects
@@
 			(project ""
 				(path "/8e13b6ca-3b5b-4f2e-83bc-fdfde26a6699/6c7faaef-a9df-4a02-8e80-f9afae2d6d46"
-					(reference "D5")
+					(reference "D6")
 					(unit 1)
 				)
@@
 	(symbol
 		(lib_id "Device:R_Potentiometer")
-		(at 218.44 85.09 180)
+		(at 218.44 83.82 0)
 		(unit 1)
 		(exclude_from_sim no)
@@
 		(dnp no)
 		(property "Reference" "RV1"
-			(at 220.726 83.82 0)
+			(at 216.154 85.09 0)
 			(effects
 				(font
@@
 		)
 		(property "Value" "10k"
-			(at 220.726 85.852 0)
+			(at 216.154 83.058 0)
 			(effects
 				(font
@@
 		)
 		(property "Footprint" "Potentiometer_THT:Potentiometer_Bourns_3296W_Vertical"
-			(at 218.44 85.09 0)
+			(at 218.44 83.82 0)
 			(effects
 				(font
@@
 		)
 		(property "Datasheet" "~"
-			(at 218.44 85.09 0)
+			(at 218.44 83.82 0)
 			(effects
 				(font
@@
 		)
 		(property "Description" "Potentiometer"
-			(at 218.44 85.09 0)
+			(at 218.44 83.82 0)
 			(effects
 				(font
@@
 		(on_board yes)
 		(dnp no)
-		(fields_autoplaced yes)
-		(property "Reference" "SW2"
-			(at 254 73.6601 90)
+		(property "Reference" "SW1"
+			(at 251.714 73.406 90)
 			(effects
 				(font
@@
 		)
 		(property "Value" "JS202011JAQN"
-			(at 254 71.1201 90)
+			(at 251.714 70.866 90)
 			(effects
 				(font
@@
 			(project ""
 				(path "/8e13b6ca-3b5b-4f2e-83bc-fdfde26a6699/6c7faaef-a9df-4a02-8e80-f9afae2d6d46"
-					(reference "SW2")
+					(reference "SW1")
 					(unit 1)
 				)
@@
 		(dnp no)
 		(fields_autoplaced yes)
-		(property "Reference" "D3"
+		(property "Reference" "D4"
 			(at 168.2947 64.4524 90)
 			(effects
@@
 			(project "LightspeedLaserDriver"
 				(path "/8e13b6ca-3b5b-4f2e-83bc-fdfde26a6699/6c7faaef-a9df-4a02-8e80-f9afae2d6d46"
-					(reference "D3")
+					(reference "D4")
 					(unit 1)
 				)

Commit message: feat(pcb): laser driver layout draft finished, add high voltage indicator LED and discharge path
Parts:
- RV1: footprint Potentiometer_THT:Potentiometer_Bourns_3296W_Vertical -> Potentiometer_SMD:Potentiometer_Bourns_3314J_Vertical
Connections:
- net FBX: no longer RV1.2
- net BOOST_NODE3: now reaches C7.1, C8.2, D3.1 (K), R5.2
- net BOOST_NODE1: now reaches C6.1, D3.2 (A), IC1.14 (SW2), IC1.16 (SW1), L1.2
- net BOOST_NODE2: now reaches C6.2, D4.1 (K), D5.2 (A)
- net at R7.1, RV1.3: now also RV1.2
Other:
- moved on the sheet: D6, R10, R6, R7, R8, R9, RV1, SW1

Commit message: feat(pcb): improve the design draft
Parts:
- C2: value 100u;100V -> 100n;100V
- C4: value 1nF;16V -> 1n;16V
- C7: value 220nF;200V -> 220n;200V
- C8: value 200nF;200V -> 220n;200V
- D6: value LED -> APTD1608LCGCK
- L1: value 74438356220 -> 7443732448100; footprint Inductor_SMD:L_Wuerth_MAPI-4020 -> Inductor_SMD_Wurth:L_Wurth_WE-LQSH-4020
- R8: value 47k -> 47k;1%
- RV1: value 10k -> 3314J-1-103G
Connections:
- net GND: now also SW1.1 (A)
- net at R8.1, R9.2, SW1.2 (B): no longer SW1.1 (A)
Other:
- note added: "Reference design: 74437324100 (10uH, 120V) Available alternative: 74438336100 (10uH, 80V, tiny) Available alternative: 74438356150 (15uH, 80V) Better alternative: 74438356220 (22uH, 80V) New replacement part: 7443732448100 (10uH, 120V) Performance alternative: 744393305220 (22uH, 120V?)"
- note removed: "Reference design: 74437324100 (10uH) Available alternative: 74438336100 (10uH, tiny) Available alternative: 74438356150 (15uH) Better alternative: 74438356220 (22uH) Performance alternative: 744393305220 (22uH)"
Changed lines of the file:
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@@
 		)
 	)
-	(text "Reference design:        74437324100  (10uH)\nAvailable alternative:     74438336100  (10uH, tiny)\nAvailable alternative:     74438356150  (15uH)\nBetter alternative:        74438356220  (22uH)\nPerformance alternative:  744393305220 (22uH)"
+	(text "Reference design:        74437324100  (10uH, 120V)\nAvailable alternative:     74438336100  (10uH, 80V, tiny)\nAvailable alternative:     74438356150  (15uH, 80V)\nBetter alternative:        74438356220  (22uH, 80V)\nNew replacement part:    7443732448100 (10uH, 120V)\nPerformance alternative:  744393305220 (22uH, 120V?)"
 		(exclude_from_sim no)
 		(at 81.788 62.484 0)
@@
 	)
 	(junction
-		(at 256.54 83.82)
-		(diameter 0)
-		(color 0 0 0 0)
-	)
-	(junction
 		(at 165.1 81.28)
 		(diameter 0)
@@
 	(wire
 		(pts
-			(xy 260.35 67.31) (xy 256.54 67.31)
-		)
-		(stroke
-			(width 0)
-			(type default)
-		)
-	)
-	(wire
-		(pts
 			(xy 154.94 92.71) (xy 154.94 95.25)
 		)
@@
 	(wire
 		(pts
-			(xy 256.54 67.31) (xy 256.54 83.82)
-		)
-		(stroke
-			(width 0)
-			(type default)
-		)
-	)
-	(wire
-		(pts
 			(xy 69.85 105.41) (xy 69.85 106.68)
 		)
@@
 	(wire
 		(pts
-			(xy 260.35 68.58) (xy 260.35 67.31)
-		)
-		(stroke
-			(width 0)
-			(type default)
-		)
-	)
-	(wire
-		(pts
 			(xy 256.54 85.09) (xy 256.54 83.82)
 		)
@@
 		)
 	)
+	(label "GND"
+		(at 260.35 68.58 90)
+		(effects
+			(font
+				(size 1.27 1.27)
+			)
+			(justify left bottom)
+		)
+	)
 	(label "EN"
 		(at 78.74 92.71 0)
@@
 			)
 		)
-		(property "Value" "1nF;16V"
+		(property "Value" "1n;16V"
 			(at 72.898 120.904 0)
 			(effects
@@
 			)
 		)
-		(property "Value" "47k"
+		(property "Value" "47k;1%"
 			(at 254 89.662 0)
 			(effects
@@
 			)
 		)
-		(property "Value" "100u;100V"
+		(property "Value" "100n;100V"
 			(at 50.292 90.17 0)
 			(effects
@@
 			)
 		)
-		(property "Value" "74438356220"
+		(property "Value" "7443732448100"
 			(at 104.14 78.74 90)
 			(effects
@@
 			)
 		)
-		(property "Footprint" "Inductor_SMD:L_Wuerth_MAPI-4020"
+		(property "Footprint" "Inductor_SMD_Wurth:L_Wurth_WE-LQSH-4020"
 			(at 104.14 81.28 0)
 			(effects
@@
 			)
 		)
-		(property "Value" "LED"
+		(property "Value" "APTD1608LCGCK"
 			(at 252.73 101.9174 90)
 			(effects
@@
 			)
 		)
-		(property "Value" "10k"
+		(property "Value" "3314J-1-103G"
 			(at 219.964 84.328 0)
 			(effects
@@
 			)
 		)
-		(property "Value" "220nF;200V"
+		(property "Value" "220n;200V"
 			(at 187.452 72.39 0)
 			(effects
@@
 			)
 		)
-		(property "Value" "200nF;200V"
+		(property "Value" "220n;200V"
 			(at 187.706 91.44 0)
 			(effects
