File: 02_PCB/LightspeedLaserDriver/LightspeedLaserDriver.kicad_pcb (KiCad board)
At the start: 2 copper layers, 57 x 32 mm, 58 parts, among them IC1 LT8365JMSE, J1 694106106102, J2 SMA, J3 Conn_01x02_Pin, J4 SMA, Q1 PJA3463_R1_00001, Q2 FMMT417TD, SW1 JS202011JAQN

Commit message: feat(pcb): laser driver V0.1 as ordered on 08.03.2026
Other:
- board text added: "Fixed Pulsewidth Avalanche Laser Driver Output adjustable between 100-260V (c) Hannes Duske 2026 V0.1"
- board text removed: "Fixed Pulsewidth Avalanche Laser Driver Output is adjustable between 100-260V (c) Hannes Duske 2026 V0.1"
Changed lines of the file:
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@@
 		(grid_origin 160 110)
 		(pcbplotparams
-			(layerselection 0x00000000_00000000_55555555_5757f5ff)
+			(layerselection 0x00000000_00000000_55555555_5755f5ff)
 			(plot_on_all_layers_selection 0x00000000_00000000_00000000_00000000)
 			(disableapertmacros no)
-			(usegerberextensions no)
-			(usegerberattributes yes)
-			(usegerberadvancedattributes yes)
-			(creategerberjobfile yes)
+			(usegerberextensions yes)
+			(usegerberattributes no)
+			(usegerberadvancedattributes no)
+			(creategerberjobfile no)
 			(dashed_line_dash_ratio 12.000000)
 			(dashed_line_gap_ratio 3.000000)
@@
 		)
 		(embedded_fonts no)
+		(model "${KICAD9_3DMODEL_DIR}/Resistor_SMD.3dshapes/R_0603_1608Metric.step"
+			(offset
+				(xyz 0 0 0)
+			)
+			(scale
+				(xyz 1 1 1)
+			)
+			(rotate
+				(xyz -0 -0 -90)
+			)
+		)
 	)
 	(footprint "Resistor_SMD:R_0805_2012Metric"
@@
 		(sheetfile "LightspeedLaserDriver.kicad_sch")
 		(attr smd)
-		(fp_line
-			(start -0.210242 -1.985)
-			(end 0.210242 -1.985)
-			(stroke
-				(width 0.12)
-				(type solid)
-			)
-			(layer "F.SilkS")
-		)
-		(fp_line
-			(start -0.210242 1.985)
-			(end 0.210242 1.985)
-			(stroke
-				(width 0.12)
-				(type solid)
-			)
-			(layer "F.SilkS")
-		)
 		(fp_rect
 			(start -1.88 -2.28)
@@
 		)
 	)
-	(gr_text "Fixed Pulsewidth\nAvalanche Laser Driver\n\nOutput is adjustable\nbetween 100-260V\n\n(c) Hannes Duske 2026\nV0.1"
+	(gr_text "Fixed Pulsewidth\nAvalanche Laser Driver\n\nOutput adjustable\nbetween 100-260V\n\n(c) Hannes Duske 2026\nV0.1"
 		(at 131.5 110 270)
 		(layer "B.SilkS")
