File: 03_PCB/LightspeedLaserDriver/DriverStage.kicad_sch (KiCad schematic)
At the start: 20 parts, among them Q2 FMMT417TD

Commit message: chore: restructure desing files in repo
Parts:
- renumbered C12 to C?, C9 to C?, C11 to C?, D7 to D?, D10 to D?, D9 to D?, D8 to D?, NT1 to NT?, Q2 to Q?, R18 to R?, R20 to R?, R16 to R?, R12 to R?, R17 to R?, R15 to R?, R14 to R?, R11 to R?, R13 to R?, R19 to R?, TR1 to TR?
Other:
- note added: "The trigger input uses a wideband RF transformer that galvannically isolates the trigger input to protect the connected signal source. This also limits the trigger pulse width (high pass) which prevents damage to the system from sustained input signals that keep the BJT turned on. The additional diode limits reverse voltage at the base that happens when the trigger signal goes from high to low."
- note removed: "The trigger input uses a wideband RF transformwe to galvannically isolate the trigger input to protect the connected signal source. This also limits the trigger pulse width which prevents damage to the system from sustained input signals that keep the BJT turned on. The additional diode limits reverse voltage at the base that happens when the trigger signal goes from high to low."
