File: 03_PCB/LightspeedLaserDriver/LightspeedLaserDriver.kicad_pcb (KiCad board)
At the start: 2 copper layers, 57 x 32 mm, 58 parts, among them IC1 LT8365JMSE, J1 694106106102, J2 SMA, J3 Conn_01x02_Pin, J4 SMA, Q1 PJA3463_R1_00001, Q2 FMMT417TD, SW1 JS202011JAQN

Commit message: chore: restructure desing files in repo
Other:
- board text added: "SENSE 100A/V 50Ω"
- board text removed: "SENSE 20A/V 50Ω"
