File: 03_PCB/AvalancheLaserDriver/DriverStage.kicad_sch (KiCad schematic)
At the start: 22 parts, among them Q2 FMMT417TD, Q3 PMBT6429-QR

Commit message: feat(pcb): laser driver V0.2 as ordered on 08.04.2026
Parts:
- R12: value 10k;1% -> 47k;1%
Other:
- company: (none) -> Hannes Duske
- title: (none) -> Driver Stage
- moved on the sheet: D9
Changed lines of the file:
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@@
 	(generator_version "9.0")
 	(paper "A4")
+	(title_block
+		(title "Driver Stage")
+		(date "2026-02-27")
+		(rev "0.2")
+		(company "Hannes Duske")
+	)
 	(text "The trigger input uses a wideband RF transformer that galvannically isolates\nthe trigger input to protect the connected signal source. This also limits\nthe trigger pulse width (high pass) which prevents damage to the system from sustained\ninput signals that keep the BJT turned on. The additional diode limits reverse\nvoltage at the base that happens when the trigger signal goes from high to low."
 		(exclude_from_sim no)
@@
 	(wire
 		(pts
-			(xy 177.8 53.34) (xy 177.8 68.58)
+			(xy 177.8 58.42) (xy 177.8 68.58)
 		)
 		(stroke
@@
 	(wire
 		(pts
-			(xy 177.8 43.18) (xy 177.8 45.72)
+			(xy 177.8 43.18) (xy 177.8 50.8)
 		)
 		(stroke
@@
 	(symbol
 		(lib_id "Device:D_Schottky")
-		(at 177.8 49.53 90)
+		(at 177.8 54.61 90)
 		(unit 1)
 		(exclude_from_sim no)
@@
 		(fields_autoplaced yes)
 		(property "Reference" "D9"
-			(at 180.34 48.5774 90)
+			(at 180.34 53.6574 90)
 			(effects
 				(font
@@
 		)
 		(property "Value" "SMD115PBQ-TP"
-			(at 180.34 51.1174 90)
+			(at 180.34 56.1974 90)
 			(effects
 				(font
@@
 		)
 		(property "Footprint" "CustomFootprints:D_SOD-323HE"
-			(at 177.8 49.53 0)
+			(at 177.8 54.61 0)
 			(effects
 				(font
@@
 		)
 		(property "Datasheet" "~"
-			(at 177.8 49.53 0)
+			(at 177.8 54.61 0)
 			(effects
 				(font
@@
 		)
 		(property "Description" "Schottky diode"
-			(at 177.8 49.53 0)
+			(at 177.8 54.61 0)
 			(effects
 				(font
@@
 			)
 		)
-		(property "Value" "10k;1%"
+		(property "Value" "47k;1%"
 			(at 110.49 39.37 90)
 			(effects

Commit message: chore(pcb): update schematic with tuned component values and update notes
Other:
- note added: "A wideband RF transformer is used for galvannic isolation of the trigger input to protect the connected signal source. This also limits the trigger pulse width (high pass) which prevents damage to the system from sustained input signals that would keep the BJT turned on. The additional diode limits reverse voltage at the BJT base that happens when the trigger signal goes from high to low. The BJT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"
- note added: "Input has 50Ω termination"
- note added: "Output reads 100A/V"
- note added: "The output pulse length roughly follows: C*V=I*t - Reference: Les Lab produced a 2ns electrical pulse with 376pF at 200V - At a constant pulse energy smaller caps with higher charging voltage yield shorter pulses than large caps with a lower voltage - We will use 200pF up to 316V Optimize design for small ESI to deliver the stored energy faster - No pulse shaping resistors - Smallest possible cap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"
- note removed: "The output pulse length roughly follows: C*V=I*t Les Lab produced a 2ns electrical pulse with 376pF at 200V We will use 200pF at 250V -> higher currents -> shorter pulse but same energy We optimize for smallest ESI to deliver the stored energy faster - No pulse shaping resistors - Smallest possible cap package with sufficient voltage rating - Multiple caps in parallel with less capacitance for ov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"
- note removed: "The trigger input uses a wideband RF transformer that galvannically isolates the trigger input to protect the connected signal source. This also limits the trigger pulse width (high pass) which prevents damage to the system from sustained input signals that keep the BJT turned on. The additional diode limits reverse voltage at the base that happens when the trigger signal goes from high to low."
- title: Driver Stage -> Avalanche Laser Driver
Changed lines of the file:
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@@
 	(paper "A4")
 	(title_block
-		(title "Driver Stage")
+		(title "Avalanche Laser Driver")
 		(date "2026-02-27")
 		(rev "0.2")
 		(company "Hannes Duske")
 	)
-	(text "The trigger input uses a wideband RF transformer that galvannically isolates\nthe trigger input to protect the connected signal source. This also limits\nthe trigger pulse width (high pass) which prevents damage to the system from sustained\ninput signals that keep the BJT turned on. The additional diode limits reverse\nvoltage at the base that happens when the trigger signal goes from high to low."
+	(text "A wideband RF transformer is used for galvannic isolation\nof the trigger input to protect the connected signal source.\nThis also limits the trigger pulse width (high pass) which\nprevents damage to the system from sustained input signals\nthat would keep the BJT turned on. The additional diode limits\nreverse voltage at the BJT base that happens when the trigger\nsignal goes from high to low.\n\nThe BJT Q3 is added to achieve consist trigger signals\nat the avalanche transistor base regardless of the voltage\nof TRIG_IN. The addition of the trigger transistor considerably\nimproved the stability of the output current pulses."
 		(exclude_from_sim no)
-		(at 89.154 165.354 0)
+		(at 105.41 161.29 0)
 		(effects
 			(font
@@
 			)
 			(justify left top)
+		)
+	)
+	(text "Input has\n50Ω termination"
+		(exclude_from_sim no)
+		(at 90.17 118.11 0)
+		(effects
+			(font
+				(size 1.27 1.27)
+			)
 		)
 	)
@@
 		)
 	)
-	(text "The output pulse length roughly follows: C*V=I*t\n\nLes Lab produced a 2ns electrical pulse with 376pF at 200V\nWe will use 200pF at 250V\n-> higher currents -> shorter pulse but same energy\n\nWe optimize for smallest ESI to deliver the stored energy faster\n- No pulse shaping resistors\n- Smallest possible cap package with sufficient voltage rating\n- Multiple caps in parallel with less capacitance for overall lower ESI\n- Optimize the layout for smallest possible current loop\n- Limit current through the charging diode, as it has 25pF capacitance\n  itself that significantly slows down the electrical pulse\n\nWould have liked to use four 47pF caps, but couldn't find any\nthat were in stock with 500V voltage rating."
+	(text "Output reads\n100A/V"
 		(exclude_from_sim no)
-		(at 14.986 165.354 0)
+		(at 227.838 61.976 0)
 		(effects
 			(font
+				(size 1.27 1.27)
+			)
+		)
+	)
+	(text "The output pulse length roughly follows: C*V=I*t\n- Reference: Les Lab produced a 2ns electrical pulse with 376pF at 200V\n- At a constant pulse energy smaller caps with higher charging voltage\n  yield shorter pulses than large caps with a lower voltage\n- We will use 200pF up to 316V\n\nOptimize design for small ESI to deliver the stored energy faster\n- No pulse shaping resistors\n- Smallest possible cap package with sufficient voltage rating\n- Multiple caps in parallel with less capacitance for overall lower ESI\n- Optimize the layout for smallest possible current loop\n  (This design has all components on one side, double sided assembly could potentially\n   have lower ESI because of smaller current loop between parallel traces)\n\nWould have liked to use four 47pF caps, but couldn't find any\nthat were in stock with 500V voltage rating."
+		(exclude_from_sim no)
+		(at 15.24 161.29 0)
+		(effects
+			(font
