File: 03_PCB/AvalancheLaserDriver/InputProtection.kicad_sch (KiCad schematic)
At the start: 9 parts, among them Q1 PJA3463_R1_00001, SW1 JS202011JAQN

Commit message: feat(pcb): laser driver V0.2 as ordered on 08.04.2026
Connections:
- no-connect marks 0 -> 1
Other:
- company: (none) -> Hannes Duske
- title: (none) -> Input Protection
Changed lines of the file:
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@@
 	(generator_version "9.0")
 	(paper "A4")
+	(title_block
+		(title "Input Protection")
+		(date "2026-02-27")
+		(rev "0.2")
+		(company "Hannes Duske")
+	)
 	(junction
 		(at 125.73 86.36)
@@
 		(color 0 0 0 0)
 	)
+	(no_connect
+		(at 189.23 88.9)
+	)
 	(wire

Commit message: chore(pcb): update schematic with tuned component values and update notes
Other:
- note added: "Input Protection"
- title: Input Protection -> Avalanche Laser Driver
Changed lines of the file:
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@@
 	(paper "A4")
 	(title_block
-		(title "Input Protection")
+		(title "Avalanche Laser Driver")
 		(date "2026-02-27")
 		(rev "0.2")
 		(company "Hannes Duske")
 	)
+	(text "Input Protection"
+		(exclude_from_sim no)
+		(at 148.336 74.422 0)
+		(effects
+			(font
+				(size 1.778 1.778)
+				(thickness 0.3556)
+				(bold yes)
+			)
+		)
+	)
 	(junction
